File: GS_controller/Hardware/GS_controller/GS_controller.kicad_pcb (KiCad board)
At the start: 4 copper layers, 82.6 x 45.1 mm, 63 parts, among them IC1 MIC5528-3.3YMT-TR, J0 0, J1 USB_C_Receptacle_USB2.0_16P, J2 0, U1 USBLC6-2SC6, U2 STM32L412CBUx, U3 NRF24L01, Y1 Crystal_GND24_Small, Y2 16MHz

Commit message: added boot resistor and made last minit changes
Parts:
- added D4: 1N5819WS, Diode_SMD:D_SOD-323, B.Cu at (156.8, 59.6)
- added H1: MountingHole, MountingHole:MountingHole_3.2mm_M3_ISO7380, F.Cu at (93.0, 49.0)
- added H2: MountingHole, MountingHole:MountingHole_3.2mm_M3_ISO7380, F.Cu at (159.0, 50.0)
- added J_BOOT1: 0, Resistor_SMD:R_0603_1608Metric, F.Cu at (125.8, 79.1)
- renumbered R18 to R1, R2 to R13, R7 to R2, R8 to R7, R1 to R8, U2 to U1, U1 to U2
Connections:
- D2 pad 1: unconnected-(D2-K-Pad1) -> Net-(D2-K)
- D2 pad 2: unconnected-(D2-A-Pad2) -> Net-(D2-A)
- J1 pad A5: unconnected-(J1-CC1-PadA5) -> Net-(J1-CC1)
- J1 pad B5: unconnected-(J1-CC2-PadB5) -> Net-(J1-CC2)
- J_VBAT1 pad 1: unconnected-(J_VBAT1-Pad1) -> Net-(U1-VBAT)
- R1 pad 2: unconnected-(D2-K-Pad1) -> Net-(D2-K)
- R13 pad 1: unconnected-(J1-CC2-PadB5) -> Net-(J1-CC2)
- R8 pad 1: unconnected-(J1-CC1-PadA5) -> Net-(J1-CC1)
- U1 pad 1: unconnected-(J_VBAT1-Pad1) -> Net-(U1-VBAT)
- U1 pad 17: (no net) -> unconnected-(U1-PA7-Pad17)
- U1 pad 18: (no net) -> unconnected-(U1-PB0-Pad18)
- U1 pad 25: (no net) -> unconnected-(U1-PB12-Pad25)
- U1 pad 29: (no net) -> unconnected-(U1-PA8-Pad29)
- U1 pad 3: (no net) -> unconnected-(U1-PC14-Pad3)
- U1 pad 38: unconnected-(D2-A-Pad2) -> Net-(D2-A)
- U1 pad 39: (no net) -> unconnected-(U1-PB3-Pad39)
- U1 pad 4: (no net) -> unconnected-(U1-PC15-Pad4)
- U1 pad 40: (no net) -> unconnected-(U1-PB4-Pad40)
- U1 pad 41: (no net) -> unconnected-(U1-PB5-Pad41)
- U1 pad 42: (no net) -> unconnected-(U1-PB6-Pad42)
- U1 pad 43: (no net) -> unconnected-(U1-PB7-Pad43)
- U1 pad 44: (no net) -> Net-(U1-PH3)
- U1 pad 45: (no net) -> unconnected-(U1-PB8-Pad45)
- U1 pad 46: (no net) -> unconnected-(U1-PB9-Pad46)
- U1 pad 7: (no net) -> unconnected-(U1-NRST-Pad7)
Routing:
- net /50 OhmRF I/O: track 1.00 -> 32.3 mm
- net GND: track 67.8 -> 81.4 mm, vias 39 -> 60
- net +5V_USB: track 3.85 -> 17.0 mm
- net 3.3V_Digi: track 36.5 -> 43.3 mm, vias 13 -> 14
- net /B_2: track 34.8 -> 41.3 mm
- net /A_2: track 38.3 -> 44.8 mm
- net unconnected-(D2-A-Pad2): track 4.71 -> 0.00 mm
- net Net-(D2-A): track 0.00 -> 4.71 mm
- net Net-(U3-VDD_PA): track 8.00 -> 3.78 mm
- net unconnected-(J_VBAT1-Pad1): track 3.01 -> 0.00 mm
- net Net-(U1-VBAT): track 0.00 -> 3.01 mm
- net unconnected-(J1-CC2-PadB5): track 2.79 -> 0.00 mm, vias 1 -> 0
- net unconnected-(J1-CC1-PadA5): track 2.79 -> 0.00 mm, vias 1 -> 0
- net Net-(J1-CC2): track 0.00 -> 2.79 mm, vias 0 -> 1
- net Net-(J1-CC1): track 0.00 -> 2.79 mm, vias 0 -> 1
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- added copper zone on In1.Cu, net 3.3V_Digi
- added copper zone on In2.Cu, net GND
