File: GS_controller/Hardware/GS_controller/Controller.kicad_sch (KiCad schematic)
At the start: 25 parts, among them J1 USB_C_Receptacle_USB2.0_16P, U1 USBLC6-2SC6, U2 STM32L412CBUx, Y1 Crystal_GND24_Small

Commit message: added boot resistor and made last minit changes
Parts:
- added D4: 1N5819WS, Diode_SMD:D_SOD-323, symbol Diode:1N5819WS
- added J_BOOT1: 0, Resistor_SMD:R_0603_1608Metric, symbol Device:R_Small
Connections:
- net +5V_USB: now also D4.2 (A)
- net GND: now also J_BOOT1.2
- net V_Bat: now also D4.1 (K)
- net at U2.44 (PH3): now also J_BOOT1.1
- no-connect marks 3 -> 2

Commit message: made order and started on cad
Parts:
- C15, C16: value TODO -> 12p
- R18, R6: value TODO -> 1k
- R5: value 10k -> 22k
- R7: value TODO -> 5.1k
- R8: value TODO -> 10k
Changed lines of the file:
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@@
 			)
 		)
-		(property "Value" "TODO"
+		(property "Value" "5.1k"
 			(at 165.1 100.33 0)
 			(effects
@@
 			)
 		)
-		(property "Value" "TODO"
+		(property "Value" "12p"
 			(at 34.544 146.558 0)
 			(effects
@@
 			)
 		)
-		(property "Value" "TODO"
+		(property "Value" "10k"
 			(at 164.846 108.204 0)
 			(effects
@@
 			)
 		)
-		(property "Value" "TODO"
+		(property "Value" "12p"
 			(at 46.736 146.558 0)
 			(effects
@@
 			)
 		)
-		(property "Value" "10k"
+		(property "Value" "22k"
 			(at 240.03 44.196 0)
 			(effects
@@
 			)
 		)
-		(property "Value" "TODO"
+		(property "Value" "1k"
 			(at 118.11 97.536 0)
 			(effects
@@
 			)
 		)
-		(property "Value" "TODO"
+		(property "Value" "1k"
 			(at 255.27 44.196 0)
 			(effects
