File: STM32_FC/Hardware/Flight_Controller/Power.kicad_sch (KiCad schematic)
At the start: 18 parts, among them IC1 LMR51420XDDCR, IC3 MIC5528-3.3YMT-TR, IC5 MIC5528-3.3YMT-TR

Commit message: made order and started on cad
Parts:
- R_FBB1: value TODO -> 13k
Changed lines of the file:
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@@
 			)
 		)
-		(property "Value" "TODO"
+		(property "Value" "13k"
 			(at 93.218 61.214 0)
 			(effects
