File: STM32_FC/Hardware/Flight_Controller/STM32L412CBUx.kicad_sch (KiCad schematic)
At the start: 26 parts, among them J1 USB_C_Receptacle_USB2.0_16P, U1 USBLC6-2SC6, U2 STM32L412CBUx, Y1 Crystal_GND24_Small

Commit message: added boot resistor and made last minit changes
Parts:
- added J2: DNC, Resistor_SMD:R_0603_1608Metric, symbol Device:R_Small
Connections:
- net GND: now also J2.2
- net USART1TX: now reaches U2.42 (PB6)
- net Boot0: now reaches U2.44 (PH3)
- net Boot0: now also J2.1
- net PB9: now reaches U2.46 (PB9)
- net PB7 renamed USART1RX
- no-connect marks 3 -> 1

Commit message: made order and started on cad
Parts:
- C15, C16: value TODO -> 12p
- R18, R6, R8: value TODO -> 1k
- R5: value 10k -> 22k
- R7: value TODO -> 5.1k
Other:
- moved on the sheet: R7, R8
Changed lines of the file:
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@@
 	)
 	(junction
-		(at 167.64 100.33)
+		(at 161.29 100.33)
 		(diameter 0)
 		(color 0 0 0 0)
@@
 	(wire
 		(pts
-			(xy 167.64 107.95) (xy 167.64 106.68)
+			(xy 161.29 107.95) (xy 161.29 106.68)
 		)
 		(stroke
@@
 	(wire
 		(pts
-			(xy 167.64 99.06) (xy 167.64 100.33)
+			(xy 161.29 99.06) (xy 161.29 100.33)
 		)
 		(stroke
@@
 	(wire
 		(pts
-			(xy 170.18 100.33) (xy 167.64 100.33)
+			(xy 163.83 100.33) (xy 161.29 100.33)
 		)
 		(stroke
@@
 	(wire
 		(pts
-			(xy 167.64 92.71) (xy 167.64 93.98)
+			(xy 161.29 92.71) (xy 161.29 93.98)
 		)
 		(stroke
@@
 	(wire
 		(pts
-			(xy 167.64 100.33) (xy 167.64 101.6)
+			(xy 161.29 100.33) (xy 161.29 101.6)
 		)
 		(stroke
@@
 		)
 	)
+	(text_box "Calculations:\nBattery\nmax 4.2V per Cell\nmax S4 batteries aka 16,8V\n-> bat_volt measurement till 20V\n\nMax voltage ADC: 3V\n-> Voltage divider of 6.66667\n\nResulution ADC uC:\n12bit -> 4096 steps\n4096 steps at 3V ~ 0,73mV/Stemp\n\nResolution V_Bat measurement:\n6,1 * 0,73mV ~ 4,453mV"
+		(exclude_from_sim no)
+		(at 175.895 87.63 0)
+		(size 37.465 33.655)
+		(stroke
+			(width -0.0001)
+			(type default)
+			(color 255 255 0 1)
+		)
+		(fill
+			(type color)
+			(color 194 194 0 1)
+		)
+		(effects
+			(font
+				(size 1.27 1.27)
+				(italic yes)
+				(color 0 0 0 1)
+			)
+			(justify left top)
+		)
+	)
 	(text "uC"
 		(exclude_from_sim no)
@@
 		)
 	)
-	(label "I2C1_SCL"
-		(at 193.04 107.95 180)
-		(fields_autoplaced yes)
-		(effects
-			(font
-				(size 1.27 1.27)
-			)
-			(justify right bottom)
-		)
-	)
 	(label "RCC_OSC_IN"
 		(at 58.42 48.26 180)
@@
 	)
 	(label "V_Bat_Div"
-		(at 170.18 100.33 0)
+		(at 163.83 100.33 0)
 		(fields_autoplaced yes)
 		(effects
@@
 		)
 	)
-	(label "I2C1_SDA"
-		(at 193.04 110.49 180)
-		(fields_autoplaced yes)
-		(effects
-			(font
-				(size 1.27 1.27)
-			)
-			(justify right bottom)
-		)
-	)
 	(label "USB_D-"
 		(at 101.6 71.12 0)
@@
 	(symbol
 		(lib_id "Device:R_Small")
-		(at 167.64 96.52 180)
+		(at 161.29 96.52 180)
 		(unit 1)
 		(exclude_from_sim no)
@@
 		(dnp no)
 		(property "Reference" "R7"
-			(at 163.83 95.758 0)
+			(at 157.48 95.758 0)
 			(effects
 				(font
@@
 			)
 		)
-		(property "Value" "TODO"
-			(at 163.83 97.79 0)
+		(property "Value" "5.1k"
+			(at 157.48 97.79 0)
 			(effects
 				(font
@@
 		)
 		(property "Footprint" "Resistor_SMD:R_0603_1608Metric"
-			(at 167.64 96.52 0)
+			(at 161.29 96.52 0)
 			(effects
 				(font
@@
 		)
 		(property "Datasheet" "~"
-			(at 167.64 96.52 0)
+			(at 161.29 96.52 0)
 			(effects
 				(font
@@
 		)
 		(property "Description" "Resistor, small symbol"
-			(at 167.64 96.52 0)
+			(at 161.29 96.52 0)
 			(effects
 				(font
@@
 			)
 		)
-		(property "Value" "TODO"
+		(property "Value" "1k"
 			(at 254 41.656 0)
 			(effects
@@
 			)
 		)
-		(property "Value" "TODO"
+		(property "Value" "12p"
 			(at 53.594 168.148 0)
 			(effects
@@
 	(symbol
 		(lib_id "power:+6V")
-		(at 167.64 92.71 0)
+		(at 161.29 92.71 0)
 		(unit 1)
 		(exclude_from_sim no)
@@
 		(fields_autoplaced yes)
 		(property "Reference" "#PWR023"
-			(at 167.64 96.52 0)
+			(at 161.29 96.52 0)
 			(effects
 				(font
@@
 		)
 		(property "Value" "V_Bat"
-			(at 167.64 87.63 0)
+			(at 161.29 87.63 0)
 			(effects
 				(font
@@
 		)
 		(property "Footprint" ""
-			(at 167.64 92.71 0)
+			(at 161.29 92.71 0)
 			(effects
 				(font
@@
 		)
 		(property "Datasheet" ""
-			(at 167.64 92.71 0)
+			(at 161.29 92.71 0)
 			(effects
 				(font
@@
 		)
 		(property "Description" "Power symbol creates a global label with name \"+6V\""
-			(at 167.64 92.71 0)
+			(at 161.29 92.71 0)
 			(effects
 				(font
@@
 			)
 		)
-		(property "Value" "10k"
+		(property "Value" "22k"
 			(at 238.76 41.656 0)
 			(effects
@@
 	(symbol
 		(lib_id "Device:R_Small")
-		(at 167.64 104.14 180)
+		(at 161.29 104.14 180)
 		(unit 1)
 		(exclude_from_sim no)
@@
 		(dnp no)
 		(property "Reference" "R8"
-			(at 163.576 103.378 0)
+			(at 157.226 103.378 0)
 			(effects
 				(font
@@
 			)
 		)
-		(property "Value" "TODO"
-			(at 163.576 105.664 0)
+		(property "Value" "1k"
+			(at 157.226 105.664 0)
 			(effects
 				(font
@@
 		)
 		(property "Footprint" "Resistor_SMD:R_0603_1608Metric"
-			(at 167.64 104.14 0)
+			(at 161.29 104.14 0)
 			(effects
 				(font
@@
 		)
 		(property "Datasheet" "~"
-			(at 167.64 104.14 0)
+			(at 161.29 104.14 0)
 			(effects
 				(font
@@
 		)
 		(property "Description" "Resistor, small symbol"
-			(at 167.64 104.14 0)
+			(at 161.29 104.14 0)
 			(effects
 				(font
@@
 			)
 		)
-		(property "Value" "TODO"
+		(property "Value" "12p"
 			(at 65.786 168.148 0)
 			(effects
@@
 			)
 		)
-		(property "Value" "TODO"
+		(property "Value" "1k"
 			(at 130.81 74.676 0)
 			(effects
@@
 	(symbol
 		(lib_id "power:GND")
-		(at 167.64 107.95 0)
+		(at 161.29 107.95 0)
 		(unit 1)
 		(exclude_from_sim no)
@@
 		(fields_autoplaced yes)
 		(property "Reference" "#PWR026"
-			(at 167.64 114.3 0)
+			(at 161.29 114.3 0)
 			(effects
 				(font
@@
 		)
 		(property "Value" "GND"
-			(at 167.64 113.03 0)
+			(at 161.29 113.03 0)
 			(effects
 				(font
@@
 		)
 		(property "Footprint" ""
-			(at 167.64 107.95 0)
+			(at 161.29 107.95 0)
 			(effects
 				(font
@@
 		)
 		(property "Datasheet" ""
-			(at 167.64 107.95 0)
+			(at 161.29 107.95 0)
 			(effects
 				(font
@@
 		)
 		(property "Description" "Power symbol creates a global label with name \"GND\" , ground"
-			(at 167.64 107.95 0)
+			(at 161.29 107.95 0)
 			(effects
 				(font
