File: STM32_FC/Hardware/Flight_Controller/Flight_Controller.kicad_pcb (KiCad board)
At the start: 4 copper layers, 51 x 50 mm, 88 parts, among them IC1 LMR51420XDDCR, IC2 ICM-42670-P, IC3 MIC5528-3.3YMT-TR, IC4 IIS2MDCTR, IC5 MIC5528-3.3YMT-TR, J1 USB_C_Receptacle_USB2.0_16P, U1 USBLC6-2SC6, U2 STM32L412CBUx, U3 VL53L0CXV0DH_1, U5 NRF24L01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

Commit message: added boot resistor and made last minit changes
Parts:
- added J2: DNC, Resistor_SMD:R_0603_1608Metric, F.Cu at (37.5, 38.4)
- moved C9 0.33 mm to (35.4, 41.3)
Connections:
- IC2 pad 12: /STM32L412CBUx/PB7 -> /STM32L412CBUx/PB9
- U2 pad 42: unconnected-(U2-PB6-Pad42) -> /STM32L412CBUx/USART1TX
- U2 pad 43: /STM32L412CBUx/PB7 -> /STM32L412CBUx/USART1RX
- U2 pad 44: unconnected-(U2-PH3-Pad44) -> /STM32L412CBUx/Boot0
- U2 pad 46: unconnected-(U2-PB9-Pad46) -> /STM32L412CBUx/PB9
Routing:
- net /STM32L412CBUx/USART1TX: track 0.00 -> 28.1 mm, vias 0 -> 2
- net /STM32L412CBUx/USART1RX: track 0.00 -> 27.7 mm, vias 0 -> 2
- net 3.3V_Digi: track 101.9 -> 123.1 mm, vias 20 -> 21
- net 3.3V_Anal: track 80.5 -> 95.7 mm, vias 8 -> 10
- net /STM32L412CBUx/PB9: track 0.00 -> 12.0 mm, vias 0 -> 2
- net /Com/50 OhmRF I/O: track 20.5 -> 32.3 mm
- net /STM32L412CBUx/PB7: track 9.73 -> 0.00 mm, vias 2 -> 0
- net /STM32L412CBUx/Boot0: track 0.00 -> 5.32 mm
- net /STM32L412CBUx/I2C1_SCL: track 22.1 -> 23.4 mm
- net GND: track 91.4 -> 92.7 mm, vias 37 -> 49
- net /STM32L412CBUx/I2C1_SDA: track 21.5 -> 22.8 mm
- net /STM32L412CBUx/ESC_SDA: track 111.0 -> 112.0 mm
- net /STM32L412CBUx/PB8: track 10.7 -> 10.1 mm
- added copper zone on In1.Cu, net GND
Other:
- board text added: "3v RX TX GN"
- board text added: "GN SC SD 3V"

Commit message: made order and started on cad
Other:
- board size 51 x 50 mm -> 50 x 50 mm
Changed lines of the file:
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@@
 		(layer "F.Mask")
-	)
-	(gr_line
-		(start 64.7 48.65)
-		(end 64.7 25.45)
-		(stroke
-			(width 0.05)
-			(type default)
-		)
-		(layer "Edge.Cuts")
 	)
 	(gr_arc
@@
 	)
 	(gr_line
-		(start 64.7 49.55)
-		(end 63.7 49.55)
-		(stroke
-			(width 0.05)
-			(type default)
-		)
-		(layer "Edge.Cuts")
-	)
-	(gr_line
-		(start 64.7 24.75)
-		(end 64.7 21.507157)
-		(stroke
-			(width 0.05)
-			(type default)
-		)
-		(layer "Edge.Cuts")
-	)
-	(gr_line
 		(start 63.7 49.55)
 		(end 63.688 60.66)
@@
 	)
 	(gr_line
-		(start 63.7 25.45)
-		(end 63.7 48.65)
-		(stroke
-			(width 0.05)
-			(type default)
-		)
-		(layer "Edge.Cuts")
-	)
-	(gr_line
 		(start 63.688 16.66)
-		(end 63.7 24.75)
-		(stroke
-			(width 0.05)
-			(type default)
-		)
-		(layer "Edge.Cuts")
-	)
-	(gr_line
-		(start 63.7 48.65)
-		(end 64.7 48.65)
-		(stroke
-			(width 0.05)
-			(type default)
-		)
-		(layer "Edge.Cuts")
-	)
-	(gr_line
-		(start 63.7 24.75)
-		(end 64.7 24.75)
-		(stroke
-			(width 0.05)
-			(type default)
-		)
-		(layer "Edge.Cuts")
-	)
-	(gr_line
-		(start 64.7 55.507157)
-		(end 64.7 49.55)
+		(end 63.7 49.55)
 		(stroke
 			(width 0.05)
@@
 		(stroke
 			(width 0.05)
-			(type default)
-		)
-		(layer "Edge.Cuts")
-	)
-	(gr_line
-		(start 63.7 25.45)
-		(end 64.7 25.45)
-		(stroke
-			(width 0.05)

Commit message: added stm32 things
Parts:
- C15, C16: value TODO -> 12p
- R18, R6, R8: value TODO -> 1k
- R5: value 10k -> 22k
- R7: value TODO -> 5.1k
- R_FBB1: value TODO -> 13k
Changed lines of the file:
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@@
 			)
 		)
-		(property "Value" "TODO"
+		(property "Value" "12p"
 			(at 0 1.16 0)
 			(layer "F.Fab")
@@
 			)
 		)
-		(property "Value" "TODO"
+		(property "Value" "12p"
 			(at 0 1.16 0)
 			(layer "F.Fab")
@@
 			)
 		)
-		(property "Value" "TODO"
+		(property "Value" "13k"
 			(at 0 1.43 90)
 			(layer "F.Fab")
@@
 			)
 		)
-		(property "Value" "TODO"
+		(property "Value" "5.1k"
 			(at 0 1.43 90)
 			(layer "F.Fab")
@@
 			)
 		)
-		(property "Value" "10k"
+		(property "Value" "22k"
 			(at 0 1.43 0)
 			(layer "F.Fab")
@@
 			)
 		)
-		(property "Value" "TODO"
+		(property "Value" "1k"
 			(at 0 1.43 0)
 			(layer "F.Fab")
@@
 			)
 		)
-		(property "Value" "TODO"
+		(property "Value" "1k"
 			(at 0 1.43 0)
 			(layer "F.Fab")
@@
 			)
 		)
-		(property "Value" "TODO"
+		(property "Value" "1k"
 			(at 0 1.43 90)
 			(layer "F.Fab")
