File: STM32_FC/Hardware/Flight_Controller/Flight_Controller.kicad_sch (KiCad schematic)
At the start: 3 parts

Commit message: added boot resistor and made last minit changes
Other:
- sheet STM32L412CBUx ports: added PB9; removed PB7
Changed lines of the file:
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@@
 	)
 	(sheet
-		(at 35.56 74.295)
+		(at 35.56 74.93)
 		(size 41.91 52.07)
 		(fields_autoplaced yes)
@@
 		)
 		(property "Sheetname" "Power"
-			(at 35.56 73.5834 0)
+			(at 35.56 74.2184 0)
 			(effects
 				(font
@@
 		)
 		(property "Sheetfile" "Power.kicad_sch"
-			(at 35.56 126.9496 0)
+			(at 35.56 127.5846 0)
 			(effects
 				(font
@@
 			)
 		)
-		(pin "PB7" bidirectional
-			(at 171.45 88.9 0)
-			(effects
-				(font
-					(size 1.27 1.27)
-				)
-				(justify right)
-			)
-		)
 		(pin "SWCLK{slash}PA14" bidirectional
 			(at 171.45 93.98 0)
@@
 			(effects
 				(font
+					(size 1.27 1.27)
+				)
+				(justify right)
+			)
+		)
+		(pin "PB9" bidirectional
+			(at 171.45 88.9 0)
+			(effects
+				(font

Commit message: made order and started on cad
Changed lines of the file:
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@@
+		)
+	)
+	(text_box "Known Design Errors:\nCom Quarz footprint is wrong\n"
+		(exclude_from_sim no)
+		(at 226.06 29.845 0)
+		(size 37.465 33.655)
+		(stroke
+			(width -0.0001)
+			(type default)
+			(color 255 255 0 1)
+		)
+		(fill
+			(type color)
+			(color 194 194 0 1)
+		)
+		(effects
+			(font
+				(size 1.27 1.27)
+				(italic yes)
+				(color 0 0 0 1)
+			)
+			(justify left top)
 		)
 	)

Commit message: added stm32 things
Changed lines of the file:
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@@
 		)
 	)
-	(text_box "Known Design Errors:\nCom Quarz footprint is wrong\n"
+	(text_box "Known Design Errors:\n- Com Quarz footprint is wrong\n- USB diode to 5V line not Vbat\n- Missing Boot0 button as well as reset\n- Battery labeling switched\n"
 		(exclude_from_sim no)
 		(at 226.06 29.845 0)
-		(size 37.465 33.655)
+		(size 46.99 17.145)
 		(stroke
 			(width -0.0001)
