File: STM32_ESC/Hardware/ESC/ESC.kicad_pcb (KiCad board)
At the start: 4 copper layers, 44 x 44 mm, 90 parts, among them IC1 IR2103STRPBF, IC2 LMR51420XDDCR, IC3 IR2103STRPBF, IC4 IR2103STRPBF, J1 USB_C_Receptacle_USB2.0_16P, Q1 IRFH8318TRPBF, Q2 BSC060P03NS3E G, Q3 BSC060P03NS3E G, Q4 IRFH8318TRPBF, Q5 IRFH8318TRPBF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

Commit message: added boot resistor and made last minit changes
Parts:
- added J_BOOT1: 0, Resistor_SMD:R_0603_1608Metric, B.Cu at (37.8, 26.8)
Connections:
- U1 pad 44: unconnected-(U1-PH3-Pad44) -> Net-(U1-PH3)
Routing:
- net GND: track 74.8 -> 78.5 mm, vias 68 -> 67
- net Net-(U1-PH3): track 0.00 -> 3.14 mm, vias 0 -> 1
- net /I2C1_CL: track 8.99 -> 8.20 mm, vias 2 -> 1
- net /I2C1_SDA: track 8.89 -> 8.77 mm, vias 2 -> 1

Commit message: made stm32 software work in vscode
Parts:
- C26, C27: value TODO -> 12p
- R11, R15, R21, R7: value TODO -> 5.1k
- R12, R16, R22, R26, R8: value TODO -> 1k
- R25: value 10k -> 22k
Changed lines of the file:
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@@
 			)
 		)
-		(property "Value" "TODO"
+		(property "Value" "1k"
 			(at 0 1.43 90)
 			(layer "F.Fab")
@@
 			)
 		)
-		(property "Value" "TODO"
+		(property "Value" "1k"
 			(at 0 1.43 90)
 			(layer "F.Fab")
@@
 			)
 		)
-		(property "Value" "TODO"
+		(property "Value" "1k"
 			(at 0 1.43 90)
 			(layer "F.Fab")
@@
 			)
 		)
-		(property "Value" "TODO"
+		(property "Value" "5.1k"
 			(at 0 1.43 90)
 			(layer "F.Fab")
@@
 			)
 		)
-		(property "Value" "TODO"
+		(property "Value" "5.1k"
 			(at 0 1.43 90)
 			(layer "F.Fab")
@@
 			)
 		)
-		(property "Value" "TODO"
+		(property "Value" "5.1k"
 			(at 0 1.43 90)
 			(layer "F.Fab")
@@
 			)
 		)
-		(property "Value" "TODO"
+		(property "Value" "12p"
 			(at 0 1.16 0)
 			(layer "F.Fab")
@@
 			)
 		)
-		(property "Value" "TODO"
+		(property "Value" "12p"
 			(at 0 1.16 0)
 			(layer "F.Fab")
@@
 			)
 		)
-		(property "Value" "TODO"
+		(property "Value" "5.1k"
 			(at 0 -1.43 0)
 			(layer "B.Fab")
@@
 			)
 		)
-		(property "Value" "TODO"
+		(property "Value" "1k"
 			(at 0 -1.43 90)
 			(layer "B.Fab")
@@
 			)
 		)
-		(property "Value" "10k"
+		(property "Value" "22k"
 			(at 0 -1.43 90)
 			(layer "B.Fab")
@@
 			)
 		)
-		(property "Value" "TODO"
+		(property "Value" "1k"
 			(at 0 -1.43 90)
 			(layer "B.Fab")
@@
 		(tags "resistor")
 		(property "Reference" "J_BOOT1"
-			(at 0 1.43 360)
+			(at 0 1.43 0)
 			(layer "B.SilkS")
 			(effects
@@
 		)
 		(property "Value" "0"
-			(at 0 -1.43 360)
+			(at 0 -1.43 0)
 			(layer "B.Fab")
 			(effects
@@
 		)
 		(fp_text user "${REFERENCE}"
-			(at 0 0 360)
+			(at 0 0 0)
 			(layer "B.Fab")
 			(effects
