File: STM32_ESC/Hardware/ESC/ESC.kicad_sch (KiCad schematic)
At the start: 90 parts, among them IC1 IR2103STRPBF, IC2 LMR51420XDDCR, IC3 IR2103STRPBF, IC4 IR2103STRPBF, J1 USB_C_Receptacle_USB2.0_16P, Q1 IRFH8318TRPBF, Q2 BSC060P03NS3E G, Q3 BSC060P03NS3E G, Q4 IRFH8318TRPBF, Q5 IRFH8318TRPBF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

Commit message: added boot resistor and made last minit changes
Parts:
- added J_BOOT1: 0, Resistor_SMD:R_0603_1608Metric, symbol Device:R_Small
Connections:
- net GND: now also J_BOOT1.2
- net at U1.44 (PH3): now also J_BOOT1.1
- no-connect marks 17 -> 16
Changed lines of the file:
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@@
 	)
 	(no_connect
-		(at 49.53 213.36)
-	)
-	(no_connect
 		(at 49.53 256.54)
 	)
@@
 	(wire
 		(pts
+			(xy 45.72 213.36) (xy 49.53 213.36)
+		)
+		(stroke
+			(width 0)
+			(type default)
+		)
+	)
+	(wire
+		(pts
 			(xy 232.41 27.94) (xy 236.22 27.94)
 		)
@@
 	(wire
 		(pts
+			(xy 38.1 213.36) (xy 40.64 213.36)
+		)
+		(stroke
+			(width 0)
+			(type default)
+		)
+	)
+	(wire
+		(pts
 			(xy 118.11 250.19) (xy 118.11 264.16)
 		)
@@
 	(wire
 		(pts
+			(xy 38.1 213.36) (xy 38.1 214.63)
+		)
+		(stroke
+			(width 0)
+			(type default)
+		)
+	)
+	(wire
+		(pts
 			(xy 201.93 223.52) (xy 209.55 223.52)
 		)
@@
 	)
 	(symbol
+		(lib_id "Device:R_Small")
+		(at 43.18 213.36 270)
+		(unit 1)
+		(exclude_from_sim no)
+		(in_bom yes)
+		(on_board yes)
+		(dnp no)
+		(property "Reference" "J_BOOT1"
+			(at 43.942 215.9 90)
+			(effects
+				(font
+					(size 1.27 1.27)
+				)
+			)
+		)
+		(property "Value" "0"
+			(at 44.704 217.17 0)
+			(effects
+				(font
+					(size 1.27 1.27)
+				)
+				(hide yes)
+			)
+		)
+		(property "Footprint" "Resistor_SMD:R_0603_1608Metric"
+			(at 43.18 213.36 0)
+			(effects
+				(font
+					(size 1.27 1.27)
+				)
+				(hide yes)
+			)
+		)
+		(property "Datasheet" "~"
+			(at 43.18 213.36 0)
+			(effects
+				(font
+					(size 1.27 1.27)
+				)
+				(hide yes)
+			)
+		)
+		(property "Description" "Resistor, small symbol"
+			(at 43.18 213.36 0)
+			(effects
+				(font
+					(size 1.27 1.27)
+				)
+				(hide yes)
+			)
+		)
+		(pin "2"
+		)
+		(pin "1"
+		)
+		(instances
+			(project "ESC"
+				(path "/a998ef63-1881-46ed-abf4-8d9591ea0fbd"
+					(reference "J_BOOT1")
+					(unit 1)
+				)
+			)
+		)
+	)
+	(symbol
 		(lib_id "power:+3V3")
 		(at 111.76 104.14 0)
@@
 					(unit 1)
 				)
+			)
+		)
+	)
+	(symbol
+		(lib_id "power:GND")
+		(at 38.1 214.63 0)
+		(unit 1)
+		(exclude_from_sim no)
+		(in_bom yes)
+		(on_board yes)
+		(dnp no)
+		(fields_autoplaced yes)
+		(property "Reference" "#PWR049"
+			(at 38.1 220.98 0)
+			(effects
+				(font
+					(size 1.27 1.27)
+				)
+				(hide yes)
+			)
+		)
+		(property "Value" "GND"
+			(at 38.1 219.71 0)
+			(effects
+				(font
+					(size 1.27 1.27)
+				)
+				(hide yes)
+			)
+		)
+		(property "Footprint" ""
+			(at 38.1 214.63 0)
+			(effects
+				(font
+					(size 1.27 1.27)
+				)
+				(hide yes)
+			)
+		)
+		(property "Datasheet" ""
+			(at 38.1 214.63 0)
+			(effects
+				(font
+					(size 1.27 1.27)
+				)
+				(hide yes)
+			)
+		)
+		(property "Description" "Power symbol creates a global label with name \"GND\" , ground"
+			(at 38.1 214.63 0)
+			(effects
+				(font
+					(size 1.27 1.27)
+				)
+				(hide yes)
+			)
+		)
+		(pin "1"
+		)
+		(instances
+			(project "ESC"
+				(path "/a998ef63-1881-46ed-abf4-8d9591ea0fbd"
+					(reference "#PWR049")
+					(unit 1)
+				)

Commit message: made order and started on cad
Parts:
- C26, C27: value TODO -> 12p
- R11, R15, R21, R7: value TODO -> 5.1k
- R12, R16, R22, R26, R8: value TODO -> 1k
- R25: value 10k -> 22k
Changed lines of the file:
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@@
 			)
 		)
-		(property "Value" "TODO"
+		(property "Value" "12p"
 			(at 108.204 260.858 0)
 			(effects
@@
 			)
 		)
-		(property "Value" "TODO"
+		(property "Value" "1k"
 			(at 119.126 204.724 0)
 			(effects
@@
 			)
 		)
-		(property "Value" "TODO"
+		(property "Value" "12p"
 			(at 120.396 260.858 0)
 			(effects
@@
 			)
 		)
-		(property "Value" "TODO"
+		(property "Value" "5.1k"
 			(at 119.38 196.85 0)
 			(effects
@@
 			)
 		)
-		(property "Value" "10k"
+		(property "Value" "22k"
 			(at 95.25 115.316 0)
 			(effects
@@
 			)
 		)
-		(property "Value" "TODO"
+		(property "Value" "1k"
 			(at 266.446 246.634 0)
 			(effects
@@
 			)
 		)
-		(property "Value" "TODO"
+		(property "Value" "1k"
 			(at 115.57 115.316 0)
 			(effects
@@
 			)
 		)
-		(property "Value" "TODO"
+		(property "Value" "5.1k"
 			(at 266.7 238.76 0)
 			(effects
@@
 			)
 		)
-		(property "Value" "TODO"
+		(property "Value" "1k"
 			(at 266.446 156.464 0)
 			(effects
@@
 			)
 		)
-		(property "Value" "TODO"
+		(property "Value" "5.1k"
 			(at 266.7 148.59 0)
 			(effects
@@
 			)
 		)
-		(property "Value" "TODO"
+		(property "Value" "5.1k"
 			(at 270.51 58.42 0)
 			(effects
@@
 			)
 		)
-		(property "Value" "TODO"
+		(property "Value" "1k"
 			(at 270.256 66.294 0)
 			(effects

Commit message: updated
Other:
- note added: "Design Errors -NMos Source/Drain Switched"
- moved on the sheet: C18, C19, C20, C21, C22, C23, C26, C27, J_BOOT1, J_VBAT1, J_VUSB1, R7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

Commit message: updated
Other:
- note added: "Design Errors -NMos Source/Drain Switched -Halfbridge Driver for 2 NMos -no Boot/Reset Buttons"
- note removed: "Design Errors -NMos Source/Drain Switched"
Changed lines of the file:
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@@
 		)
 	)
-	(text "Design Errors\n -NMos Source/Drain Switched"
+	(text "Design Errors\n -NMos Source/Drain Switched\n -Halfbridge Driver for 2 NMos\n -no Boot/Reset Buttons\n"
 		(exclude_from_sim no)
 		(at 304.8 138.176 0)
