File: STM32_ESC/Hardware/ESC_V1.1/ESC.kicad_pcb (KiCad board)
At the start: 4 copper layers, 44 x 44 mm, 91 parts, among them IC1 IR2103STRPBF, IC2 LMR51420XDDCR, IC3 IR2103STRPBF, IC4 IR2103STRPBF, J1 USB_C_Receptacle_USB2.0_16P, Q1 BSC060P03NS3E G, Q2 BSC060P03NS3E G, Q3 BSC060P03NS3E G, Q4 BSC060P03NS3E G, Q5 IRFH8318TRPBF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

Commit message: updated
Parts:
- C18, C22: moved to F.Cu
- moved C22 12.0 mm to (47.5, 35.8)
- moved C18 3.87 mm to (31.2, 34.0), turned to 0 degrees
Connections:
- D6 pad 2: +3V3 -> /Status_LED
- U1 pad 2: unconnected-(U1-PC13-Pad2) -> /Status_LED
Routing:
- net V_Bat: track 126.0 -> 19.1 mm, vias 1 -> 11
- net +3V3: track 127.9 -> 37.0 mm
- net GND: track 58.8 -> 45.5 mm, vias 37 -> 32
- net /Status_LED: track 0.00 -> 9.27 mm
- net +5V_USB: track 37.2 -> 38.4 mm
- added copper zone on In1.Cu, net +3V3
- added copper zone on In1.Cu, net GND
- added copper zone on In2.Cu, net GND
- added copper zone on B.Cu, net V_Bat
- added copper zone on F.Cu, net V_Bat
