File: STM32_ESC/Hardware/ESC_V1.1/ESCV1_1.kicad_pcb (KiCad board)
At the start: 4 copper layers, 44 x 44 mm, 90 parts, among them IC1 IR2103STRPBF, IC2 LMR51420XDDCR, IC3 IR2103STRPBF, IC4 IR2103STRPBF, J1 USB_C_Receptacle_USB2.0_16P, Q1 IRFH8318TRPBF, Q2 IRFH8318TRPBF, Q3 IRFH8318TRPBF, Q4 IRFH8318TRPBF, Q5 IRFH8318TRPBF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

Commit message: updated
Routing:
- net /boot: track 29.9 -> 32.3 mm
Changed lines of the file:
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@@
+	)
+	(segment
+		(start 54.8 43.3)
+		(end 54.8 45.025)
+		(width 0.2)
+		(layer "F.Cu")
+		(net "/boot")
+	)
+	(segment
+		(start 54.8 45.025)
+		(end 54.325 45.5)
+		(width 0.2)
+		(layer "F.Cu")
+		(net "/boot")
 	)
 	(segment

Commit message: updated
Routing:
- net GND: track 48.7 -> 64.4 mm, vias 39 -> 41
- net +3V3: track 37.3 -> 38.4 mm, vias 10 -> 11
Changed lines of the file:
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@@
+	)
+	(segment
+		(start 48.275 35.75)
+		(end 48.925 36.4)
+		(width 0.2)
+		(layer "F.Cu")
+		(net "GND")
 	)
 	(segment
@@
 	)
 	(segment
+		(start 41.65 39.95)
+		(end 42.8 38.8)
+		(width 0.2)
+		(layer "F.Cu")
+		(net "GND")
+	)
+	(segment
+		(start 48.925 36.4)
+		(end 49.815738 36.4)
+		(width 0.2)
+		(layer "F.Cu")
+		(net "GND")
+	)
+	(segment
 		(start 44.125 35.5625)
 		(end 44.125 36.695)
+		(width 0.2)
+		(layer "F.Cu")
+		(net "GND")
+	)
+	(segment
+		(start 49.815738 36.4)
+		(end 49.920737 36.504999)
 		(width 0.2)
 		(layer "F.Cu")
@@
 	)
 	(segment
+		(start 39.25 39.95)
+		(end 41.65 39.95)
+		(width 0.2)
+		(layer "F.Cu")
+		(net "GND")
+	)
+	(segment
 		(start 46.545 29.875)
 		(end 45.3125 29.875)
@@
 	)
 	(via
+		(at 39.6 38.2)
+		(size 0.6)
+		(drill 0.3)
+		(layers "F.Cu" "B.Cu")
+		(net "GND")
+	)
+	(via
 		(at 61 55.5)
 		(size 0.6)
@@
 		)
 		(filling no)
+		(net "GND")
+	)
+	(via
+		(at 42.8 38.8)
+		(size 0.6)
+		(drill 0.3)
+		(layers "F.Cu" "B.Cu")
 		(net "GND")
 	)
@@
 	)
 	(segment
+		(start 36.37 38.8)
+		(end 39 38.8)
+		(width 0.2)
+		(layer "B.Cu")
+		(net "GND")
+	)
+	(segment
+		(start 48.8 38.625)
+		(end 48.8 37.625736)
+		(width 0.2)
+		(layer "B.Cu")
+		(net "GND")
+	)
+	(segment
+		(start 48.8 37.625736)
+		(end 49.920737 36.504999)
+		(width 0.2)
+		(layer "B.Cu")
+		(net "GND")
+	)
+	(segment
+		(start 28.505 37.505)
+		(end 28 37)
+		(width 0.2)
+		(layer "B.Cu")
+		(net "GND")
+	)
+	(segment
 		(start 54.505 40.188)
 		(end 55.588 40.188)
@@
 	)
 	(segment
+		(start 28.505 40.188)
+		(end 28.505 37.505)
+		(width 0.2)
+		(layer "B.Cu")
+		(net "GND")
+	)
+	(segment
+		(start 39 38.8)
+		(end 39.6 38.2)
+		(width 0.2)
+		(layer "B.Cu")
+		(net "GND")
+	)
+	(segment
+		(start 36.195 38.625)
+		(end 36.37 38.8)
+		(width 0.2)
+		(layer "B.Cu")
+		(net "GND")
+	)
+	(segment
 		(start 29.5 21.25)
 		(end 29.5 21.975)
@@
 	)
 	(segment
+		(start 46.9 34.7)
+		(end 46.725 34.875)
+		(width 0.4)
+		(layer "F.Cu")
+		(net "+3V3")
+	)
+	(segment
 		(start 29.848988 47.270869)
 		(end 30.025619 47.4475)
@@
 	)
 	(segment
+		(start 46.725 34.875)
+		(end 46.725 35.75)
+		(width 0.4)
+		(layer "F.Cu")
+		(net "+3V3")
+	)
+	(segment
 		(start 46.03 35.75)
 		(end 46.725 35.75)
@@
 	)
 	(segment
+		(start 46.9 34.698527)
+		(end 46.9 34.7)
+		(width 0.4)
+		(layer "F.Cu")
+		(net "+3V3")
+	)
+	(segment
 		(start 21 36.45)
 		(end 20.8 36.65)
@@
 		(net "+3V3")
 	)
+	(via
+		(at 46.9 34.698527)
+		(size 0.6)
+		(drill 0.3)
+		(layers "F.Cu" "B.Cu")
+		(net "+3V3")
+	)

Commit message: updated
Parts:
- D1, D2, D3, D4: footprint Diode_SMD:D_SOD-323 -> Diode_SMD:D_SOD-323_HandSoldering
- moved J1 1.22 mm to (59.2, 30.6)
Routing:
- net GND: track 64.4 -> 66.7 mm, vias 41 -> 42
- net Net-(J1-CC1): track 3.58 -> 4.87 mm
- net /USB_D+: track 11.5 -> 12.7 mm
- net /USB_D-: track 12.1 -> 13.2 mm
- net /nGate_C: track 15.4 -> 16.2 mm
Other:
- board text added: "Fynn Gewiese"
