File: STM32_ESC/Hardware/ESC_V1.1/ESCV1_1.kicad_sch (KiCad schematic)
At the start: 91 parts, among them IC1 IR2103STRPBF, IC2 LMR51420XDDCR, IC3 IR2103STRPBF, IC4 IR2103STRPBF, J1 USB_C_Receptacle_USB2.0_16P, Q1 BSC060P03NS3E G, Q2 BSC060P03NS3E G, Q3 BSC060P03NS3E G, Q4 BSC060P03NS3E G, Q5 IRFH8318TRPBF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

Commit message: updated
Parts:
- removed Q1, Q2, Q3, Q4, Q6, Q7: BSC060P03NS3E G, ESC_footrpints:BSC060P03NS3EG, symbol Simulation_SPICE:PMOS
- removed Q5: IRFH8318TRPBF, ESC_footrpints:BSC054N04NSGATMA1, symbol Simulation_SPICE:NMOS
- removed U2: USBLC6-2SC6, Package_TO_SOT_SMD:SOT-23-6, symbol Power_Protection:USBLC6-2SC6
- added Q1, Q2, Q3, Q4, Q5, Q6, Q8: IRFH8318TRPBF, ESC_footrpints:BSC054N04NSGATMA1, symbol ESC_Library:IRFH8318TRPBF
- C24, C25, U6: value ~ -> (none)
Connections:
- net Phase_A: now also Q5.S, Q6.D
- net Phase_B: now also Q3.S, Q4.D
- net Phase_C: now also Q1.S, Q2.D
- net USB_D+: now also J1.A6 (D+), J1.B6 (D+)
- net USB_D-: now also J1.A7 (D-), J1.B7 (D-)
- net V_Bat: now also Q1.D, Q3.D, Q5.D, Q8.S
- net V_Bat_raw: now also Q8.D
- net nGate_A: now also Q5.G
- net nGate_B: now also Q3.G
- net nGate_C: now also Q1.G
- net pGate_A: now also Q6.G
- net pGate_B: now also Q4.G
- net pGate_C: now also Q2.G
- net at R19.1, U5.3 (+): now also Q2.S
- net at R13.1, U4.3 (+): now also Q4.S
- net at C28.1, R23.1, R24.2: now also Q8.G
- net at R1.1, U3.3 (+): now also Q6.S

Commit message: updated
Other:
- note added: "Design Fixes -NMos Source/Drain Switched -Halfbridge Driver for 2 NMos -no Boot/Reset Buttons Design Errors -wrong Diode Footprint"
- note removed: "Design Errors -NMos Source/Drain Switched -Halfbridge Driver for 2 NMos -no Boot/Reset Buttons -wrong Diode Footprint"
Changed lines of the file:
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@@
 		)
 	)
-	(text "Design Errors\n -NMos Source/Drain Switched\n -Halfbridge Driver for 2 NMos\n -no Boot/Reset Buttons\n -wrong Diode Footprint\n\n"
+	(text "Design Fixes\n -NMos Source/Drain Switched\n -Halfbridge Driver for 2 NMos\n -no Boot/Reset Buttons\nDesign Errors\n -wrong Diode Footprint\n\n"
 		(exclude_from_sim no)
-		(at 303.784 140.462 0)
+		(at 301.498 142.748 0)
 		(effects
 			(font

Commit message: updated
Parts:
- C16, C2, C8: footprint CAPAE660X550N -> (none)
- D1, D2, D3, D4: footprint Diode_SMD:D_SOD-323 -> Diode_SMD:D_SOD-323_HandSoldering
- IC1, IC3, IC4: footprint SOIC127P600X175-8N -> (none)
- IC2: footprint SOT95P280X110-6N -> (none)
- L2: footprint XAL5050822MEC -> (none)
Changed lines of the file:
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@@
 			)
 		)
-		(property "Footprint" "SOT95P280X110-6N"
+		(property "Footprint" ""
 			(at 349.25 146.99 0)
 			(hide yes)
@@
 			)
 		)
-		(property "Footprint" "Diode_SMD:D_SOD-323"
+		(property "Footprint" "Diode_SMD:D_SOD-323_HandSoldering"
 			(at 175.26 208.915 0)
 			(hide yes)
@@
 			)
 		)
-		(property "Footprint" "SOIC127P600X175-8N"
+		(property "Footprint" ""
 			(at 185.42 143.18 0)
 			(hide yes)
@@
 			)
 		)
-		(property "Footprint" "XAL5050822MEC"
+		(property "Footprint" ""
 			(at 364.49 54.61 0)
 			(hide yes)
@@
 			)
 		)
-		(property "Footprint" "CAPAE660X550N"
+		(property "Footprint" ""
 			(at 236.22 31.75 0)
 			(hide yes)
@@
 			)
 		)
-		(property "Footprint" "Diode_SMD:D_SOD-323"
+		(property "Footprint" "Diode_SMD:D_SOD-323_HandSoldering"
 			(at 309.245 46.99 0)
 			(hide yes)
@@
 			)
 		)
-		(property "Footprint" "CAPAE660X550N"
+		(property "Footprint" ""
 			(at 236.22 212.09 0)
 			(hide yes)
@@
 			)
 		)
-		(property "Footprint" "Diode_SMD:D_SOD-323"
+		(property "Footprint" "Diode_SMD:D_SOD-323_HandSoldering"
 			(at 175.26 28.575 0)
 			(hide yes)
@@
 			)
 		)
-		(property "Footprint" "SOIC127P600X175-8N"
+		(property "Footprint" ""
 			(at 185.42 233.35 0)
 			(hide yes)
@@
 			)
 		)
-		(property "Footprint" "SOIC127P600X175-8N"
+		(property "Footprint" ""
 			(at 185.42 323.52 0)
 			(hide yes)
@@
 			)
 		)
-		(property "Footprint" "Diode_SMD:D_SOD-323"
+		(property "Footprint" "Diode_SMD:D_SOD-323_HandSoldering"
 			(at 175.26 118.745 0)
 			(hide yes)
@@
 			)
 		)
-		(property "Footprint" "CAPAE660X550N"
+		(property "Footprint" ""
 			(at 236.22 121.92 0)
 			(hide yes)
