File: STM32_ESC/Hardware/ESC_V1/ESC.kicad_sch (KiCad schematic)
At the start: 91 parts, among them IC1 IR2103STRPBF, IC2 LMR51420XDDCR, IC3 IR2103STRPBF, IC4 IR2103STRPBF, J1 USB_C_Receptacle_USB2.0_16P, Q1 IRFH8318TRPBF, Q2 BSC060P03NS3E G, Q3 BSC060P03NS3E G, Q4 IRFH8318TRPBF, Q5 IRFH8318TRPBF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

Commit message: updated
Other:
- note added: "Design Errors -NMos Source/Drain Switched -Halfbridge Driver for 2 NMos -no Boot/Reset Buttons -wrong Diode Footprint"
- note removed: "Design Errors -NMos Source/Drain Switched -Halfbridge Driver for 2 NMos -no Boot/Reset Buttons"
Changed lines of the file:
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@@
 		)
 	)
-	(text "Design Errors\n -NMos Source/Drain Switched\n -Halfbridge Driver for 2 NMos\n -no Boot/Reset Buttons\n"
+	(text "Design Errors\n -NMos Source/Drain Switched\n -Halfbridge Driver for 2 NMos\n -no Boot/Reset Buttons\n -wrong Diode Footprint\n\n"
 		(exclude_from_sim no)
 		(at 304.8 138.176 0)

Commit message: updated
Parts:
- removed Q1, Q4, Q8: IRFH8318TRPBF, ESC_footrpints:BSC054N04NSGATMA1, symbol Simulation_SPICE:NMOS
- removed Q2, Q3, Q7: BSC060P03NS3E G, ESC_footrpints:BSC060P03NS3EG, symbol Simulation_SPICE:PMOS
- C24, C25, U6: value ~ -> (none)
